File: gps10mhz.sch (EAGLE design)
At the start: 28 parts, among them IC2 7803.3, IC3 CD74HC132E, U1 BB3553AM

Commit message: up
Parts:
- added C13, C14, C15, C16: 0.01uf, rcl:C-USC0805
Connections:
- net +15V: now also C14.1
- net -15V: now also C13.1
- net 0V: now also C13.2, C14.2
- net 10MHZ_IN: now also C15.2
- net 10MHZ_OUT: now also C16.1
- net IN: now also C15.1
- net OUT: now also C16.2
Other:
- moved on the sheet: R1, R2
Changed lines of the file:
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@@
 <part name="LED1" library="led" library_urn="urn:adsk.eagle:library:259" deviceset="TLLR4400" device="" package3d_urn="urn:adsk.eagle:package:15797/1"/>
 <part name="GND20" library="supply1" library_urn="urn:adsk.eagle:library:371" deviceset="0V" device=""/>
+<part name="C13" library="rcl" library_urn="urn:adsk.eagle:library:334" deviceset="C-US" device="C0805" package3d_urn="urn:adsk.eagle:package:23617/2" value="0.01uf"/>
+<part name="GND21" library="supply1" library_urn="urn:adsk.eagle:library:371" deviceset="0V" device=""/>
+<part name="C14" library="rcl" library_urn="urn:adsk.eagle:library:334" deviceset="C-US" device="C0805" package3d_urn="urn:adsk.eagle:package:23617/2" value="0.01uf"/>
+<part name="GND22" library="supply1" library_urn="urn:adsk.eagle:library:371" deviceset="0V" device=""/>
+<part name="C15" library="rcl" library_urn="urn:adsk.eagle:library:334" deviceset="C-US" device="C0805" package3d_urn="urn:adsk.eagle:package:23617/2" value="0.01uf"/>
+<part name="C16" library="rcl" library_urn="urn:adsk.eagle:library:334" deviceset="C-US" device="C0805" package3d_urn="urn:adsk.eagle:package:23617/2" value="0.01uf"/>
 </parts>
 <sheets>
@@
 </instance>
 <instance part="P+1" gate="1" x="30.48" y="27.94" smashed="yes">
-<attribute name="VALUE" x="27.94" y="22.86" size="1.778" layer="96" rot="R90"/>
+<attribute name="VALUE" x="35.56" y="25.4" size="1.778" layer="96" rot="R90"/>
 </instance>
 <instance part="P-1" gate="1" x="40.64" y="27.94" smashed="yes" rot="R180">
@@
 </instance>
 <instance part="C5" gate="G$1" x="22.86" y="38.1" smashed="yes" rot="R270">
-<attribute name="NAME" x="15.875" y="34.544" size="1.778" layer="95" rot="R270"/>
+<attribute name="NAME" x="23.495" y="42.164" size="1.778" layer="95" rot="R270"/>
 <attribute name="VALUE" x="18.669" y="37.084" size="1.778" layer="96" rot="R270"/>
 </instance>
@@
 <attribute name="VALUE" x="64.516" y="38.989" size="1.778" layer="96"/>
 </instance>
-<instance part="R1" gate="G$1" x="25.4" y="33.02" smashed="yes" rot="R90">
-<attribute name="NAME" x="23.9014" y="29.21" size="1.778" layer="95" rot="R90"/>
-<attribute name="VALUE" x="28.702" y="29.21" size="1.778" layer="96" rot="R90"/>
-</instance>
-<instance part="R2" gate="G$1" x="55.88" y="33.02" smashed="yes" rot="R90">
-<attribute name="NAME" x="54.3814" y="29.21" size="1.778" layer="95" rot="R90"/>
-<attribute name="VALUE" x="64.77" y="31.242" size="1.778" layer="96" rot="R180"/>
+<instance part="R1" gate="G$1" x="25.4" y="25.4" smashed="yes" rot="R90">
+<attribute name="NAME" x="23.9014" y="21.59" size="1.778" layer="95" rot="R90"/>
+<attribute name="VALUE" x="18.542" y="16.51" size="1.778" layer="96" rot="R90"/>
+</instance>
+<instance part="R2" gate="G$1" x="55.88" y="25.4" smashed="yes" rot="R90">
+<attribute name="NAME" x="54.3814" y="21.59" size="1.778" layer="95" rot="R90"/>
+<attribute name="VALUE" x="64.77" y="23.622" size="1.778" layer="96" rot="R180"/>
 </instance>
 <instance part="SV1" gate="G$1" x="60.96" y="86.36" smashed="yes">
@@
 <attribute name="VALUE" x="51.435" y="76.2" size="1.778" layer="96"/>
 </instance>
-<instance part="GND7" gate="1" x="55.88" y="25.4" smashed="yes">
-<attribute name="VALUE" x="53.975" y="22.86" size="1.778" layer="96"/>
+<instance part="GND7" gate="1" x="55.88" y="15.24" smashed="yes">
+<attribute name="VALUE" x="53.975" y="12.7" size="1.778" layer="96"/>
 </instance>
 <instance part="GND8" gate="1" x="68.58" y="78.74" smashed="yes">
 <attribute name="VALUE" x="66.675" y="76.2" size="1.778" layer="96"/>
 </instance>
-<instance part="GND9" gate="1" x="25.4" y="25.4" smashed="yes">
-<attribute name="VALUE" x="23.495" y="22.86" size="1.778" layer="96"/>
+<instance part="GND9" gate="1" x="25.4" y="15.24" smashed="yes">
+<attribute name="VALUE" x="23.495" y="12.7" size="1.778" layer="96"/>
 </instance>
 <instance part="GND10" gate="1" x="116.84" y="60.96" smashed="yes">
@@
 <instance part="GND20" gate="1" x="137.16" y="5.08" smashed="yes">
 <attribute name="VALUE" x="135.255" y="2.54" size="1.778" layer="96"/>
+</instance>
+<instance part="C13" gate="G$1" x="99.06" y="45.72" smashed="yes">
+<attribute name="NAME" x="100.076" y="46.355" size="1.778" layer="95"/>
+<attribute name="VALUE" x="100.076" y="41.529" size="1.778" layer="96"/>
+</instance>
+<instance part="GND21" gate="1" x="99.06" y="38.1" smashed="yes">
+<attribute name="VALUE" x="97.155" y="35.56" size="1.778" layer="96"/>
+</instance>
+<instance part="C14" gate="G$1" x="10.16" y="53.34" smashed="yes">
+<attribute name="NAME" x="11.176" y="53.975" size="1.778" layer="95"/>
+<attribute name="VALUE" x="11.176" y="49.149" size="1.778" layer="96"/>
+</instance>
+<instance part="GND22" gate="1" x="10.16" y="45.72" smashed="yes">
+<attribute name="VALUE" x="8.255" y="43.18" size="1.778" layer="96"/>
+</instance>
+<instance part="C15" gate="G$1" x="22.86" y="30.48" smashed="yes" rot="R270">
+<attribute name="NAME" x="23.495" y="34.544" size="1.778" layer="95" rot="R270"/>
+<attribute name="VALUE" x="13.589" y="34.544" size="1.778" layer="96" rot="R270"/>
+</instance>
+<instance part="C16" gate="G$1" x="60.96" y="30.48" smashed="yes" rot="R270">
+<attribute name="NAME" x="61.595" y="29.464" size="1.778" layer="95" rot="R270"/>
+<attribute name="VALUE" x="56.769" y="29.464" size="1.778" layer="96" rot="R270"/>
 </instance>
 </instances>
@@
 <pinref part="R2" gate="G$1" pin="1"/>
 <pinref part="GND7" gate="1" pin="0V"/>
-<junction x="55.88" y="27.94"/>
+<wire x1="55.88" y1="17.78" x2="55.88" y2="20.32" width="0.1524" layer="91"/>
+<junction x="55.88" y="20.32"/>
+<junction x="55.88" y="17.78"/>
 </segment>
 <segment>
@@
 <pinref part="R1" gate="G$1" pin="1"/>
 <pinref part="GND9" gate="1" pin="0V"/>
-<junction x="25.4" y="27.94"/>
+<wire x1="25.4" y1="17.78" x2="25.4" y2="20.32" width="0.1524" layer="91"/>
+<junction x="25.4" y="17.78"/>
+<junction x="25.4" y="20.32"/>
 </segment>
 <segment>
@@
 <pinref part="GND20" gate="1" pin="0V"/>
 <junction x="137.16" y="7.62"/>
+</segment>
+<segment>
+<pinref part="C13" gate="G$1" pin="2"/>
+<pinref part="GND21" gate="1" pin="0V"/>
+<junction x="99.06" y="40.64"/>
+</segment>
+<segment>
+<pinref part="C14" gate="G$1" pin="2"/>
+<pinref part="GND22" gate="1" pin="0V"/>
+<junction x="10.16" y="48.26"/>
 </segment>
 </net>
@@
 <junction x="17.78" y="55.88"/>
 <label x="7.62" y="55.88" size="1.778" layer="95"/>
+<pinref part="C14" gate="G$1" pin="1"/>
+<wire x1="17.78" y1="55.88" x2="10.16" y2="55.88" width="0.1524" layer="91"/>
+<junction x="10.16" y="55.88"/>
 </segment>
 <segment>
@@
 <junction x="99.06" y="48.26"/>
 <label x="101.6" y="48.26" size="1.778" layer="95"/>
+<pinref part="C13" gate="G$1" pin="1"/>
 </segment>
 <segment>
@@
 <pinref part="U1" gate="A" pin="OUTA"/>
 <wire x1="33.02" y1="48.26" x2="30.48" y2="48.26" width="0.1524" layer="91"/>
-<wire x1="30.48" y1="48.26" x2="30.48" y2="38.1" width="0.1524" layer="91"/>
-<wire x1="30.48" y1="38.1" x2="55.88" y2="38.1" width="0.1524" layer="91"/>
+<wire x1="30.48" y1="48.26" x2="30.48" y2="33.02" width="0.1524" layer="91"/>
+<junction x="33.02" y="48.26"/>
+<label x="35.56" y="35.56" size="1.778" layer="95"/>
 <pinref part="C6" gate="G$1" pin="2"/>
+<junction x="55.88" y="38.1"/>
 <pinref part="R2" gate="G$1" pin="2"/>
-<junction x="55.88" y="38.1"/>
-<junction x="33.02" y="48.26"/>
-<label x="38.1" y="38.1" size="1.778" layer="95"/>
+<wire x1="55.88" y1="30.48" x2="55.88" y2="33.02" width="0.1524" layer="91"/>
+<wire x1="55.88" y1="33.02" x2="55.88" y2="38.1" width="0.1524" layer="91"/>
+<wire x1="30.48" y1="33.02" x2="55.88" y2="33.02" width="0.1524" layer="91"/>
+<junction x="55.88" y="33.02"/>
+<pinref part="C16" gate="G$1" pin="2"/>
+<junction x="55.88" y="30.48"/>
 </segment>
 </net>
@@
 <pinref part="C5" gate="G$1" pin="1"/>
 <pinref part="R1" gate="G$1" pin="2"/>
-<junction x="25.4" y="38.1"/>
+<junction x="25.4" y="30.48"/>
 <junction x="33.02" y="53.34"/>
 <label x="22.86" y="43.18" size="1.778" layer="95"/>
+<wire x1="25.4" y1="38.1" x2="25.4" y2="30.48" width="0.1524" layer="91"/>
+<wire x1="25.4" y1="30.48" x2="25.4" y2="38.1" width="0.1524" layer="91"/>
+<pinref part="C15" gate="G$1" pin="1"/>
+<junction x="25.4" y="38.1"/>
 </segment>
 </net>
@@
 <junction x="63.5" y="38.1"/>
 <junction x="71.12" y="38.1"/>
+<pinref part="C16" gate="G$1" pin="1"/>
+<wire x1="63.5" y1="38.1" x2="63.5" y2="30.48" width="0.1524" layer="91"/>
+<junction x="63.5" y="30.48"/>
 </segment>
 <segment>
@@
 <junction x="17.78" y="38.1"/>
 <junction x="5.08" y="38.1"/>
+<pinref part="C15" gate="G$1" pin="2"/>
+<wire x1="17.78" y1="30.48" x2="17.78" y2="38.1" width="0.1524" layer="91"/>
+<junction x="17.78" y="30.48"/>
 </segment>
 <segment>
@@
 <pinref part="R4" gate="G$1" pin="2"/>
 <junction x="99.06" y="76.2"/>
-<pinref part="R4" gate="G$1" pin="2"/>
 <wire x1="116.84" y1="76.2" x2="104.14" y2="76.2" width="0.1524" layer="91"/>
 <pinref part="TP1" gate="G$1" pin="TP"/>

Commit message: up
Parts:
- added R6: 470, rcl:R-US_R1206
Connections:
- net N$2 renamed D1
- net N$3 renamed D2
- net N$4 renamed D3
- net 0V: now also R6.1
- net TTL: now also R6.2
Changed lines of the file:
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@@
 <part name="C15" library="rcl" library_urn="urn:adsk.eagle:library:334" deviceset="C-US" device="C0805" package3d_urn="urn:adsk.eagle:package:23617/2" value="0.01uf"/>
 <part name="C16" library="rcl" library_urn="urn:adsk.eagle:library:334" deviceset="C-US" device="C0805" package3d_urn="urn:adsk.eagle:package:23617/2" value="0.01uf"/>
+<part name="R6" library="rcl" library_urn="urn:adsk.eagle:library:334" deviceset="R-US_" device="R1206" package3d_urn="urn:adsk.eagle:package:23540/2" value="470"/>
+<part name="GND23" library="supply1" library_urn="urn:adsk.eagle:library:371" deviceset="0V" device=""/>
 </parts>
 <sheets>
@@
 <attribute name="VALUE" x="56.769" y="29.464" size="1.778" layer="96" rot="R270"/>
 </instance>
+<instance part="R6" gate="G$1" x="109.22" y="55.88" smashed="yes" rot="R90">
+<attribute name="NAME" x="107.7214" y="52.07" size="1.778" layer="95" rot="R90"/>
+<attribute name="VALUE" x="112.522" y="52.07" size="1.778" layer="96" rot="R90"/>
+</instance>
+<instance part="GND23" gate="1" x="109.22" y="48.26" smashed="yes">
+<attribute name="VALUE" x="107.315" y="45.72" size="1.778" layer="96"/>
+</instance>
 </instances>
 <busses>
@@
 <pinref part="GND22" gate="1" pin="0V"/>
 <junction x="10.16" y="48.26"/>
+</segment>
+<segment>
+<pinref part="R6" gate="G$1" pin="1"/>
+<pinref part="GND23" gate="1" pin="0V"/>
+<junction x="109.22" y="50.8"/>
 </segment>
 </net>
@@
 <junction x="142.24" y="76.2"/>
 </segment>
-</net>
-<net name="N$2" class="1">
+<segment>
+<wire x1="109.22" y1="60.96" x2="101.6" y2="60.96" width="0.1524" layer="91"/>
+<pinref part="R6" gate="G$1" pin="2"/>
+<junction x="109.22" y="60.96"/>
+<junction x="101.6" y="60.96"/>
+<label x="101.6" y="58.42" size="1.778" layer="95"/>
+</segment>
+</net>
+<net name="D1" class="1">
 <segment>
 <wire x1="129.54" y1="40.64" x2="124.46" y2="40.64" width="0.1524" layer="91"/>
@@
 <junction x="111.76" y="66.04"/>
 <junction x="116.84" y="66.04"/>
-</segment>
-</net>
-<net name="N$3" class="1">
+<label x="111.76" y="63.5" size="1.778" layer="95"/>
+</segment>
+</net>
+<net name="D2" class="1">
 <segment>
 <wire x1="144.78" y1="40.64" x2="149.86" y2="40.64" width="0.1524" layer="91"/>
@@
 <junction x="142.24" y="63.5"/>
 <junction x="147.32" y="63.5"/>
-</segment>
-</net>
-<net name="N$4" class="1">
+<label x="144.78" y="60.96" size="1.778" layer="95"/>
+</segment>
+</net>
+<net name="D3" class="1">
 <segment>
 <wire x1="144.78" y1="43.18" x2="149.86" y2="43.18" width="0.1524" layer="91"/>
@@
 <junction x="142.24" y="71.12"/>
 <junction x="147.32" y="71.12"/>
-</segment>
-</net>
+<label x="144.78" y="68.58" size="1.778" layer="95"/>
+</segment>
+</net>

Commit message: up
Parts:
- added C17: 10uf, rcl:C-USC0805
- added C18, C20, C21: 1000pf, rcl:C-USC0805
- added C19: 0.1uf, rcl:C-USC0805
- added R7: 100, rcl:R-US_R1206
- C10: value 0.1uf -> 1000pf
- C12: value 10uf -> 0.1uf
Connections:
- new net BIASV: C18.1, C19.1, R3.2, R7.2
- net +15V: now also C21.1
- net +3V3: now also C17.1, R7.1; no longer R3.2
- net -15V: now also C20.1
- net 0V: now also C17.2, C18.2, C19.2, C20.2, C21.2
Changed lines of the file:
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@@
 <part name="TP5" library="testpad" library_urn="urn:adsk.eagle:library:385" deviceset="PTR1" device="PAD1-13" package3d_urn="urn:adsk.eagle:package:27946/1"/>
 <part name="C9" library="rcl" library_urn="urn:adsk.eagle:library:334" deviceset="C-US" device="C0805" package3d_urn="urn:adsk.eagle:package:23617/2" value="0.1uf"/>
-<part name="C10" library="rcl" library_urn="urn:adsk.eagle:library:334" deviceset="C-US" device="C0805" package3d_urn="urn:adsk.eagle:package:23617/2" value="0.1uf"/>
+<part name="C10" library="rcl" library_urn="urn:adsk.eagle:library:334" deviceset="C-US" device="C0805" package3d_urn="urn:adsk.eagle:package:23617/2" value="1000pf"/>
 <part name="C11" library="rcl" library_urn="urn:adsk.eagle:library:334" deviceset="C-US" device="C0805" package3d_urn="urn:adsk.eagle:package:23617/2" value="10uf"/>
 <part name="GND16" library="supply1" library_urn="urn:adsk.eagle:library:371" deviceset="0V" device=""/>
 <part name="GND17" library="supply1" library_urn="urn:adsk.eagle:library:371" deviceset="0V" device=""/>
 <part name="GND18" library="supply1" library_urn="urn:adsk.eagle:library:371" deviceset="0V" device=""/>
-<part name="C12" library="rcl" library_urn="urn:adsk.eagle:library:334" deviceset="C-US" device="C0805" package3d_urn="urn:adsk.eagle:package:23617/2" value="10uf"/>
+<part name="C12" library="rcl" library_urn="urn:adsk.eagle:library:334" deviceset="C-US" device="C0805" package3d_urn="urn:adsk.eagle:package:23617/2" value="0.1uf"/>
 <part name="GND19" library="supply1" library_urn="urn:adsk.eagle:library:371" deviceset="0V" device=""/>
 <part name="IC3" library="CD74HC132E" deviceset="CD74HC132E" device=""/>
@@
 <part name="R6" library="rcl" library_urn="urn:adsk.eagle:library:334" deviceset="R-US_" device="R1206" package3d_urn="urn:adsk.eagle:package:23540/2" value="470"/>
 <part name="GND23" library="supply1" library_urn="urn:adsk.eagle:library:371" deviceset="0V" device=""/>
+<part name="C17" library="rcl" library_urn="urn:adsk.eagle:library:334" deviceset="C-US" device="C0805" package3d_urn="urn:adsk.eagle:package:23617/2" value="10uf"/>
+<part name="R7" library="rcl" library_urn="urn:adsk.eagle:library:334" deviceset="R-US_" device="R1206" package3d_urn="urn:adsk.eagle:package:23540/2" value="100"/>
+<part name="C18" library="rcl" library_urn="urn:adsk.eagle:library:334" deviceset="C-US" device="C0805" package3d_urn="urn:adsk.eagle:package:23617/2" value="1000pf"/>
+<part name="C19" library="rcl" library_urn="urn:adsk.eagle:library:334" deviceset="C-US" device="C0805" package3d_urn="urn:adsk.eagle:package:23617/2" value="0.1uf"/>
+<part name="GND24" library="supply1" library_urn="urn:adsk.eagle:library:371" deviceset="0V" device=""/>
+<part name="GND25" library="supply1" library_urn="urn:adsk.eagle:library:371" deviceset="0V" device=""/>
+<part name="GND26" library="supply1" library_urn="urn:adsk.eagle:library:371" deviceset="0V" device=""/>
+<part name="C20" library="rcl" library_urn="urn:adsk.eagle:library:334" deviceset="C-US" device="C0805" package3d_urn="urn:adsk.eagle:package:23617/2" value="1000pf"/>
+<part name="C21" library="rcl" library_urn="urn:adsk.eagle:library:334" deviceset="C-US" device="C0805" package3d_urn="urn:adsk.eagle:package:23617/2" value="1000pf"/>
+<part name="GND27" library="supply1" library_urn="urn:adsk.eagle:library:371" deviceset="0V" device=""/>
+<part name="GND28" library="supply1" library_urn="urn:adsk.eagle:library:371" deviceset="0V" device=""/>
 </parts>
 <sheets>
@@
 <attribute name="VALUE" x="107.315" y="45.72" size="1.778" layer="96"/>
 </instance>
+<instance part="C17" gate="G$1" x="172.72" y="76.2" smashed="yes">
+<attribute name="NAME" x="173.736" y="76.835" size="1.778" layer="95"/>
+<attribute name="VALUE" x="173.736" y="72.009" size="1.778" layer="96"/>
+</instance>
+<instance part="R7" gate="G$1" x="119.38" y="99.06" smashed="yes" rot="R180">
+<attribute name="NAME" x="123.19" y="97.5614" size="1.778" layer="95" rot="R180"/>
+<attribute name="VALUE" x="123.19" y="102.362" size="1.778" layer="96" rot="R180"/>
+</instance>
+<instance part="C18" gate="G$1" x="104.14" y="96.52" smashed="yes">
+<attribute name="NAME" x="105.156" y="97.155" size="1.778" layer="95"/>
+<attribute name="VALUE" x="102.616" y="89.789" size="1.778" layer="96"/>
+</instance>
+<instance part="C19" gate="G$1" x="111.76" y="96.52" smashed="yes">
+<attribute name="NAME" x="112.776" y="97.155" size="1.778" layer="95"/>
+<attribute name="VALUE" x="112.776" y="89.789" size="1.778" layer="96"/>
+</instance>
+<instance part="GND24" gate="1" x="104.14" y="88.9" smashed="yes">
+<attribute name="VALUE" x="102.235" y="86.36" size="1.778" layer="96"/>
+</instance>
+<instance part="GND25" gate="1" x="111.76" y="88.9" smashed="yes">
+<attribute name="VALUE" x="109.855" y="86.36" size="1.778" layer="96"/>
+</instance>
+<instance part="GND26" gate="1" x="172.72" y="68.58" smashed="yes">
+<attribute name="VALUE" x="170.815" y="66.04" size="1.778" layer="96"/>
+</instance>
+<instance part="C20" gate="G$1" x="88.9" y="45.72" smashed="yes">
+<attribute name="NAME" x="89.916" y="46.355" size="1.778" layer="95"/>
+<attribute name="VALUE" x="89.916" y="41.529" size="1.778" layer="96"/>
+</instance>
+<instance part="C21" gate="G$1" x="2.54" y="53.34" smashed="yes">
+<attribute name="NAME" x="3.556" y="53.975" size="1.778" layer="95"/>
+<attribute name="VALUE" x="3.556" y="49.149" size="1.778" layer="96"/>
+</instance>
+<instance part="GND27" gate="1" x="2.54" y="45.72" smashed="yes">
+<attribute name="VALUE" x="0.635" y="43.18" size="1.778" layer="96"/>
+</instance>
+<instance part="GND28" gate="1" x="88.9" y="38.1" smashed="yes">
+<attribute name="VALUE" x="86.995" y="35.56" size="1.778" layer="96"/>
+</instance>
 </instances>
 <busses>
@@
 <pinref part="GND23" gate="1" pin="0V"/>
 <junction x="109.22" y="50.8"/>
+</segment>
+<segment>
+<pinref part="C18" gate="G$1" pin="2"/>
+<pinref part="GND24" gate="1" pin="0V"/>
+<junction x="104.14" y="91.44"/>
+</segment>
+<segment>
+<pinref part="C19" gate="G$1" pin="2"/>
+<pinref part="GND25" gate="1" pin="0V"/>
+<junction x="111.76" y="91.44"/>
+</segment>
+<segment>
+<pinref part="C17" gate="G$1" pin="2"/>
+<pinref part="GND26" gate="1" pin="0V"/>
+<junction x="172.72" y="71.12"/>
+</segment>
+<segment>
+<pinref part="C21" gate="G$1" pin="2"/>
+<pinref part="GND27" gate="1" pin="0V"/>
+<junction x="2.54" y="48.26"/>
+</segment>
+<segment>
+<pinref part="C20" gate="G$1" pin="2"/>
+<pinref part="GND28" gate="1" pin="0V"/>
+<junction x="88.9" y="40.64"/>
 </segment>
 </net>
@@
 <wire x1="17.78" y1="55.88" x2="10.16" y2="55.88" width="0.1524" layer="91"/>
 <junction x="10.16" y="55.88"/>
+<pinref part="C21" gate="G$1" pin="1"/>
+<wire x1="2.54" y1="55.88" x2="10.16" y2="55.88" width="0.1524" layer="91"/>
+<junction x="2.54" y="55.88"/>
 </segment>
 <segment>
@@
 <label x="101.6" y="48.26" size="1.778" layer="95"/>
 <pinref part="C13" gate="G$1" pin="1"/>
+<pinref part="C20" gate="G$1" pin="1"/>
 </segment>
 <segment>
@@
 <pinref part="IC3" gate="G$1" pin="VCC"/>
 <junction x="142.24" y="78.74"/>
-</segment>
-<segment>
-<wire x1="99.06" y1="86.36" x2="106.68" y2="86.36" width="0.1524" layer="91"/>
-<pinref part="R3" gate="G$1" pin="2"/>
-<junction x="99.06" y="86.36"/>
-<junction x="106.68" y="86.36"/>
-<label x="104.14" y="88.9" size="1.778" layer="95"/>
+<wire x1="162.56" y1="78.74" x2="172.72" y2="78.74" width="0.1524" layer="91"/>
+<pinref part="C17" gate="G$1" pin="1"/>
+<junction x="172.72" y="78.74"/>
 </segment>
 <segment>
@@
 <junction x="109.22" y="78.74"/>
 <junction x="116.84" y="78.74"/>
+</segment>
+<segment>
+<wire x1="124.46" y1="99.06" x2="129.54" y2="99.06" width="0.1524" layer="91"/>
+<pinref part="R7" gate="G$1" pin="1"/>
+<junction x="124.46" y="99.06"/>
+<junction x="129.54" y="99.06"/>
+<label x="132.08" y="99.06" size="1.778" layer="95"/>
 </segment>
 </net>
@@
 </segment>
 </net>
+<net name="BIASV" class="2">
+<segment>
+<pinref part="R7" gate="G$1" pin="2"/>
+<pinref part="C19" gate="G$1" pin="1"/>
+<wire x1="114.3" y1="99.06" x2="111.76" y2="99.06" width="0.1524" layer="91"/>
+<pinref part="C18" gate="G$1" pin="1"/>
+<wire x1="104.14" y1="99.06" x2="111.76" y2="99.06" width="0.1524" layer="91"/>
+<junction x="111.76" y="99.06"/>
+<pinref part="R3" gate="G$1" pin="2"/>
+<wire x1="99.06" y1="86.36" x2="99.06" y2="99.06" width="0.1524" layer="91"/>
+<wire x1="104.14" y1="99.06" x2="99.06" y2="99.06" width="0.1524" layer="91"/>
+<junction x="104.14" y="99.06"/>
+<junction x="99.06" y="86.36"/>
+<junction x="114.3" y="99.06"/>
+</segment>
+</net>

Commit message: up
Parts:
- added C22: 10uf, rcl:C-USC0805
Connections:
- net 0V: now also C22.2
- net BIASV: now also C22.1
Changed lines of the file:
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@@
 <part name="GND27" library="supply1" library_urn="urn:adsk.eagle:library:371" deviceset="0V" device=""/>
 <part name="GND28" library="supply1" library_urn="urn:adsk.eagle:library:371" deviceset="0V" device=""/>
+<part name="C22" library="rcl" library_urn="urn:adsk.eagle:library:334" deviceset="C-US" device="C0805" package3d_urn="urn:adsk.eagle:package:23617/2" value="10uf"/>
+<part name="GND29" library="supply1" library_urn="urn:adsk.eagle:library:371" deviceset="0V" device=""/>
 </parts>
 <sheets>
@@
 <attribute name="VALUE" x="86.995" y="35.56" size="1.778" layer="96"/>
 </instance>
+<instance part="C22" gate="G$1" x="91.44" y="101.6" smashed="yes">
+<attribute name="NAME" x="92.456" y="102.235" size="1.778" layer="95"/>
+<attribute name="VALUE" x="92.456" y="97.409" size="1.778" layer="96"/>
+</instance>
+<instance part="GND29" gate="1" x="91.44" y="93.98" smashed="yes">
+<attribute name="VALUE" x="89.535" y="91.44" size="1.778" layer="96"/>
+</instance>
 </instances>
 <busses>
@@
 <pinref part="GND28" gate="1" pin="0V"/>
 <junction x="88.9" y="40.64"/>
+</segment>
+<segment>
+<pinref part="C22" gate="G$1" pin="2"/>
+<pinref part="GND29" gate="1" pin="0V"/>
+<junction x="91.44" y="96.52"/>
 </segment>
 </net>
@@
 <junction x="99.06" y="86.36"/>
 <junction x="114.3" y="99.06"/>
-</segment>
-</net>
+<pinref part="C22" gate="G$1" pin="1"/>
+<wire x1="91.44" y1="104.14" x2="99.06" y2="104.14" width="0.1524" layer="91"/>
+<wire x1="99.06" y1="104.14" x2="99.06" y2="99.06" width="0.1524" layer="91"/>
+<junction x="99.06" y="99.06"/>
+<junction x="91.44" y="104.14"/>
+</segment>
+</net>
